Commit message: Trying to construct map, but stuck at use_sim_time

File: src/my_create_map_webots/resource/MyCreate.urdf (robot description, URDF)
Before this commit: robot /home/jordenhuang/ROS2-Project/src/my_create_map_webots/resource/MyCreate.urdf, 22 links, 21 joints
Joints:
- joint base_link_bumper_left_joint: origin xyz=0 0 0 rpy=1.570806 0.000006 -0.843867 -> xyz=0 0 -0.000003 rpy=1.570806 0.000006 -0.843867
- joint base_link_bumper_right_joint: origin xyz=0 0 0 rpy=1.570792 0.000011 -2.297729 -> xyz=0 0 -0.000003 rpy=1.570792 0.000011 -2.297729
- joint left wheel motor: origin xyz=-0.0062 0 -0.014 rpy=0 0 0 -> xyz=-0.0062 0 -0.014 rpy=0 -0.000002 0
- joint right wheel motor: origin xyz=-0.0062 0.1359 -0.014 rpy=0 0 0 -> xyz=-0.0062 0.1359 -0.014 rpy=0 -0.000002 0

Commit message: Adjust params of rtabmap and rtabmap_odometry

File: src/my_create_map_webots/resource/MyCreate.urdf (robot description, URDF)
Before this commit: robot /home/jordenhuang/ROS2-Project/src/my_create_map_webots/resource/MyCreate.urdf, 22 links, 21 joints
Joints:
- joint base_link_camera_left_joint: origin xyz=0.17 0.05 0.05 rpy=-1.570796 0.261799 -1.570796 -> xyz=0.125 0.05 0.065 rpy=-1.570796 0 -1.570796
- joint base_link_camera_right_joint: origin xyz=0.17 -0.05 0.05 rpy=-1.570796 0.261799 -1.570796 -> xyz=0.17 -0.05 0.05 rpy=-1.570796 0 -1.570796

Commit message: 15 degree tilt camera

File: src/my_create_map_webots/resource/MyCreate.urdf (robot description, URDF)
Before this commit: robot /home/jordenhuang/ROS2-Project/src/my_create_map_webots/resource/MyCreate.urdf, 22 links, 21 joints
Links:
- added link camera_left_optical_frame
- added link camera_right_optical_frame
Joints:
- added joint camera_left_to_optical_joint: type fixed, parent camera_left, child camera_left_optical_frame, origin xyz=0 0 0 rpy=-1.570796 0 -1.570796
- added joint camera_right_to_optical_joint: type fixed, parent camera_right, child camera_right_optical_frame, origin xyz=0 0 0 rpy=-1.570796 0 -1.570796
- joint base_link_camera_left_joint: origin xyz=0.125 0.05 0.065 rpy=-1.570796 0 -1.570796 -> xyz=0.125 0.05 0.065 rpy=0.0 0.261799 0.0
- joint base_link_camera_right_joint: origin xyz=0.17 -0.05 0.05 rpy=-1.570796 0 -1.570796 -> xyz=0.17 -0.05 0.05 rpy=0.0 0.261799 0.0

Commit message: 改了我也不知道什麼作用的參數

File: src/my_create_map_webots/resource/MyCreate.urdf (robot description, URDF)
Before this commit: robot /home/jordenhuang/ROS2-Project/src/my_create_map_webots/resource/MyCreate.urdf, 24 links, 23 joints
Joints:
- joint base_link_camera_left_joint: origin xyz=0.125 0.05 0.065 rpy=0.0 0.261799 0.0 -> xyz=0.17 0.05 0.05 rpy=0.0 0 0.0
- joint base_link_camera_right_joint: origin xyz=0.17 -0.05 0.05 rpy=0.0 0.261799 0.0 -> xyz=0.17 -0.05 0.05 rpy=0.0 0 0.0

Commit message: 改了些參數，好像好一點，但還是很多點在地板下

File: src/my_create_map_webots/resource/MyCreate.urdf (robot description, URDF)
Before this commit: robot /home/jordenhuang/ROS2-Project/src/my_create_map_webots/resource/MyCreate.urdf, 24 links, 23 joints
Links:
- added link base_footprint
Joints:
- added joint base_joint: type fixed, parent base_link, child base_footprint, origin xyz=0 0 -0.05 rpy=0 0 0
- joint base_link_camera_left_joint: origin xyz=0.17 0.05 0.05 rpy=0.0 0 0.0 -> xyz=0.17 0.05 0.05 rpy=0.0 0.261799 0.0
- joint base_link_camera_right_joint: origin xyz=0.17 -0.05 0.05 rpy=0.0 0 0.0 -> xyz=0.17 -0.05 0.05 rpy=0.0 0.261799 0.0
